File: StrawberryV1.kicad_pcb (KiCad board)
At the start: 2 copper layers, 34 x 34 mm, 36 parts, among them J1 USB_C_Receptacle_USB2.0_16P, J2 Conn_01x05_Pin, U1 ESP32-C3FH4, U2 ICM-20948, U3 MAX30102, U5 LP5907MFX-3.3, U6 MCP73831-2-MC, U7 LP5907MFX-1.8

Commit message: update PCB unfinished
Parts:
- removed J2: Conn_01x05_Pin, Connector_JST:JST_XH_B5B-XH-A_1x05_P2.50mm_Vertical
- added J3: Conn_01x05_Pin, Connector_PinSocket_2.54mm:PinSocket_1x05_P2.54mm_Vertical, F.Cu at (109.0, 71.5)
- R1, R10, R11, R2, R3, R4, R5, R6, R7, R8, R9: footprint Resistor_SMD:R_0201_0603Metric -> Resistor_SMD:R_0603_1608Metric
- moved U7 48.5 mm to (89.8, 58.2), turned to 180 degrees
- moved R7 47.2 mm to (100.5, 59.4), turned to 90 degrees
- moved R6 46.5 mm to (98.0, 59.4), turned to 90 degrees
- moved R5 46.1 mm to (95.5, 59.4), turned to 90 degrees
- moved U5 44.9 mm to (94.2, 54.8), turned to 90 degrees
- moved C6 44.2 mm to (94.5, 51.0)
- moved R4 43.4 mm to (85.2, 73.5), turned to 90 degrees
- moved R2 43.2 mm to (81.8, 73.9), turned to 90 degrees
- moved U2 43.2 mm to (101.8, 55.8)
- moved R3 43.2 mm to (83.5, 73.8), turned to 90 degrees
- moved R11 42.0 mm to (94.8, 69.8), turned to 90 degrees
- moved R8 40.1 mm to (90.5, 75.4), turned to 90 degrees
- moved C3 37.0 mm to (106.5, 52.2)
- moved C4 37.0 mm to (106.5, 54.8)
- moved C5 37.0 mm to (106.5, 57.3)
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Connections:
- net /1p8 renamed +1V8
- C1 pad 1: ETRODE+ -> +3V3
- C10 pad 1: ETRODE+ -> +3V3
- C12 pad 1: ETRODE+ -> +3V3
- C13 pad 1: ETRODE+ -> +3V3
- C14 pad 1: ETRODE+ -> +3V3
- C3 pad 1: ETRODE+ -> +3V3
- C7 pad 1: ETRODE+ -> +3V3
- C8 pad 1: ETRODE+ -> +3V3
- C9 pad 1: ETRODE+ -> +3V3
- R10 pad 1: AREAD -> +3V3
- R5 pad 1: ETRODE+ -> +3V3
- R6 pad 2: ETRODE+ -> +3V3
- R7 pad 1: ETRODE+ -> +3V3
- U1 pad 10: AREAD -> +3V3
- U1 pad 11: ETRODE+ -> +3V3
- U1 pad 17: ETRODE+ -> +3V3
- U1 pad 18: ETRODE+ -> +3V3
- U1 pad 2: ETRODE+ -> +3V3
- U1 pad 3: ETRODE+ -> +3V3
- U1 pad 31: ETRODE+ -> +3V3
- U1 pad 32: ETRODE+ -> +3V3
- U2 pad 13: ETRODE+ -> +3V3
- U3 pad 10: ETRODE+ -> +3V3
- U3 pad 9: ETRODE+ -> +3V3
- U5 pad 5: ETRODE+ -> +3V3
- U7 pad 1: ETRODE+ -> +3V3
- U7 pad 3: ETRODE+ -> +3V3
Routing:
- net GND: track 0.00 -> 39.6 mm, vias 0 -> 5
- net +1V8: track 0.00 -> 24.9 mm, vias 0 -> 2
- net D+: track 0.00 -> 20.3 mm, vias 0 -> 2
- net D-: track 0.00 -> 18.9 mm
- net +3V3: track 0.00 -> 18.3 mm, vias 0 -> 2
- net SCL: track 0.00 -> 2.33 mm
- net SDA: track 0.00 -> 2.03 mm
Other:
- board size 34 x 34 mm -> 30 x 30 mm

Commit message: PCB almost done
Parts:
- added TP1: TestPoint, Connector_PinHeader_2.54mm:PinHeader_1x01_P2.54mm_Vertical, F.Cu at (100.0, 82.0)
- added TP2: TestPoint, Connector_PinHeader_2.54mm:PinHeader_1x01_P2.54mm_Vertical, F.Cu at (95.5, 82.0)
- D1: footprint LED_SMD:LED_0402_1005Metric -> LED_SMD:LED_0603_1608Metric
- moved R10 10.8 mm to (99.5, 78.5), turned to -90 degrees
- moved C11 8.73 mm to (107.5, 75.5)
- moved C12 8.38 mm to (106.0, 77.0), turned to 180 degrees
- moved R8 7.99 mm to (98.0, 78.2), turned to -90 degrees
- moved C7 7.61 mm to (98.0, 55.5), turned to -90 degrees
- moved C2 7.12 mm to (86.5, 59.5), turned to 90 degrees
- moved R4 6.43 mm to (91.5, 72.0), turned to -90 degrees
- moved C15 5.80 mm to (91.0, 76.5), turned to 180 degrees
- moved R2 5.33 mm to (87.0, 73.0), turned to -90 degrees
- moved D1 5.11 mm to (97.5, 75.0)
- moved R3 5.06 mm to (88.5, 73.0), turned to -90 degrees
- moved C1 4.32 mm to (90.0, 55.5), turned to 180 degrees
- moved C16 4.30 mm to (91.0, 78.0), turned to 180 degrees
- moved C3 3.76 mm to (106.3, 56.0)
- moved U6 3.68 mm to (95.0, 77.9)
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Connections:
- C12 pad 1: +3V3 -> GND
- C12 pad 2: GND -> +3V3
- R10 pad 1: +3V3 -> AREAD
- R5 pad 2: Net-(U1-EN) -> NRST
- U1 pad 10: +3V3 -> AREAD
- U1 pad 7: Net-(U1-EN) -> NRST
Routing:
- net GND: track 39.6 -> 132.6 mm, vias 5 -> 9
- net +3V3: track 18.3 -> 81.4 mm, vias 2 -> 9
- net NRST: track 0.00 -> 28.3 mm, vias 0 -> 3
- net CHGIN: track 0.00 -> 27.9 mm, vias 0 -> 4
- net Net-(J1-SHIELD): track 0.00 -> 20.6 mm
- net AREAD: track 0.00 -> 18.2 mm, vias 0 -> 3
- net Net-(U1-GP8[BOOT]): track 0.00 -> 17.2 mm, vias 0 -> 2
- net Net-(U1-GP2[BOOT]): track 0.00 -> 16.0 mm, vias 0 -> 2
- net RX: track 0.00 -> 14.9 mm, vias 0 -> 1
- net TX: track 0.00 -> 14.5 mm, vias 0 -> 3
- net BOOT: track 0.00 -> 14.3 mm
- net SDA: track 2.03 -> 15.0 mm, vias 0 -> 2
- net VBAT: track 0.00 -> 13.0 mm, vias 0 -> 2
- net +1V8: track 24.9 -> 34.9 mm, vias 2 -> 4
- net SCL: track 2.33 -> 11.8 mm, vias 0 -> 2
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Other:
- board size 30 x 30 mm -> 30 x 32.5 mm
- board text added: "Ari"
