File: StrawberryV1.kicad_sch (KiCad schematic)
At the start: 26 parts, among them J1 USB_C_Receptacle_USB2.0_16P, J3 Conn_01x03_Pin, J4 Conn_01x03_Pin, U1 ESP32-C3FH4, U2 ICM-20948, U3 MAX30102, U4 LP3982ILD-1.8, U5 AMS1117-3.3

Commit message: finished schematic
Parts:
- removed J3, J4: Conn_01x03_Pin, symbol Connector:Conn_01x03_Pin
- removed L1: L, symbol Device:L
- removed R1: 100, symbol Device:R
- removed U4: LP3982ILD-1.8, Package_SON:WSON-8-1EP_3x2.5mm_P0.5mm_EP1.2x1.5mm_PullBack_ThermalVias, symbol Regulator_Linear:LP3982ILD-1.8
- removed U5: AMS1117-3.3, Package_TO_SOT_SMD:SOT-223-3_TabPin2, symbol Regulator_Linear:AMS1117-3.3
- added C13, C14: 100n, Capacitor_SMD:C_0603_1608Metric, symbol Device:C_Small
- added C15, C16: 4.7u, Capacitor_SMD:C_0603_1608Metric, symbol Device:C_Small
- added D1: LED, LED_SMD:LED_0402_1005Metric, symbol Device:LED
- added J2: Conn_01x05_Pin, Connector_JST:JST_XH_B5B-XH-A_1x05_P2.50mm_Vertical, symbol Connector:Conn_01x05_Pin
- added R1, R11: 4.7k, Resistor_SMD:R_0201_0603Metric, symbol Device:R_Small
- added R10: 180k, Resistor_SMD:R_0201_0603Metric, symbol Device:R_Small
- added R6, R7: 10k, Resistor_SMD:R_0201_0603Metric, symbol Device:R_Small
- added R8: 30k, Resistor_SMD:R_0201_0603Metric, symbol Device:R_Small
- added R9: 470, Resistor_SMD:R_0201_0603Metric, symbol Device:R_Small
- added U5: LP5907MFX-3.3, Package_TO_SOT_SMD:SOT-23-5, symbol Regulator_Linear:LP5907MFX-3.3
- added U6: MCP73831-2-MC, Package_DFN_QFN:DFN-8-1EP_3x2mm_P0.5mm_EP1.7x1.4mm, symbol Battery_Management:MCP73831-2-MC
- added U7: LP5907MFX-1.8, Package_TO_SOT_SMD:SOT-23-5, symbol Regulator_Linear:LP5907MFX-1.8
- C1: value 2.2u -> 1u; footprint (none) -> Capacitor_SMD:C_0603_1608Metric
- C10: value 10u -> 100n; footprint (none) -> Capacitor_SMD:C_0603_1608Metric
- C11, C12, C3, C4, C5, C8, C9: footprint (none) -> Capacitor_SMD:C_0603_1608Metric
- C2: value 33n -> 1u; footprint (none) -> Capacitor_SMD:C_0603_1608Metric
- C6, C7: value C_Small -> 1u; footprint (none) -> Capacitor_SMD:C_0603_1608Metric
- R2, R3, R4, R5: footprint (none) -> Resistor_SMD:R_0201_0603Metric
- U1: footprint yume:Yu-QFN-32-5x5-0.5-EP-3.7x3.7 -> kicad libs:Yu-QFN-32-5x5-0.5-EP-3.7x3.7
Connections:
- net +3.3V: now also C9.1, U1.11 (VDD3P3_RTC), U1.17 (VDD3P3_CPU), U1.18 (VDD_SPI/GPIO11), U1.2 (VDD3P3), U1.3 (VDD3P3), U1.31 (VDDA), U1.32 (VDDA), C13.1, C14.1, R6.2, R7.1, U5.5 (OUT), U7.1 (IN), U7.3 (EN)
- net 1p8: now also C2.1, R1.1, R11.1, U7.5 (OUT)
- net GND: now also C13.2, C14.2, C15.2, C16.2, J2.1 (Pin_1), R10.2, R8.2, U5.2 (GND), U6.6 (V_{SS}), U7.2 (GND)
- net RX: now also J2.3 (Pin_3)
- net SCL: now also R1.2
- net SDA: now also R11.2
- net TX: now also J2.2 (Pin_2)
- net AREAD: now reaches U1.10 (MTDI/GP5)
- net AREAD: now also R10.1
- net +5VD renamed CHGIN
- net CHGIN: now also C15.1, D1.2 (A), U6.1 (V_{DD}), U6.2 (V_{DD}); no longer C6.1
- net BOOT_0: no longer names the net of U1.6 (GP2[BOOT])
- net BOOT_0: now also R6.1
- net BOOT_1: no longer names the net of U1.14 (GP8[BOOT])
- net BOOT_1: now also R7.2
- net BOOT_2 renamed BOOT
- net BOOT: now also J2.4 (Pin_4)
- new net: R8.1, U6.8 (PROG)
- new net: D1.1 (K), R9.1
- new net: R9.2, U6.5 (STAT)
- new net NRST: J2.5 (Pin_5)
- new net VBAT: C16.1, C6.1, U5.1 (IN), U5.3 (EN), U6.3 (V_{BAT}), U6.4 (V_{BAT})
Other:
- note added: "+VBAT to +3V3 LDO"
- note added: "Battery Management (BMIC) Battery: lp361122"
- note added: "Skin Hydration Electrodes"
- note removed: "+5V to +3V3 LDO"
- moved on the sheet: C2, C3, C4, C5, C6, C7, C8, C9, R5, U1, U2

Commit message: update PCB unfinished
Parts:
- removed J2: Conn_01x05_Pin, Connector_JST:JST_XH_B5B-XH-A_1x05_P2.50mm_Vertical, symbol Connector:Conn_01x05_Pin
- added J3: Conn_01x05_Pin, Connector_PinSocket_2.54mm:PinSocket_1x05_P2.54mm_Vertical, symbol Connector:Conn_01x05_Pin
- R1, R10, R11, R2, R3, R4, R5, R6, R7, R8, R9: footprint Resistor_SMD:R_0201_0603Metric -> Resistor_SMD:R_0603_1608Metric
Connections:
- net AREAD is gone; now on net +3.3V: R10.1, U1.10 (MTDI/GP5)
- net BOOT: now also J3.4 (Pin_4)
- net GND: now also J3.1 (Pin_1)
- net NRST: now also J3.5 (Pin_5)
- net RX: now also J3.3 (Pin_3)
- net TX: now also J3.2 (Pin_2)
- net 1p8 renamed +1V8

Commit message: PCB almost done
Parts:
- added TP1, TP2: TestPoint, Connector_PinHeader_2.54mm:PinHeader_1x01_P2.54mm_Vertical, symbol Connector:TestPoint
- D1: footprint LED_SMD:LED_0402_1005Metric -> LED_SMD:LED_0603_1608Metric
Connections:
- net +3.3V: now also C12.2, TP2.1; no longer C12.1, R10.1, U1.10 (MTDI/GP5)
- net GND: now also C12.1; no longer C12.2
- net NRST: now also R5.2, U1.7 (EN)
- new net AREAD: R10.1, TP1.1, U1.10 (MTDI/GP5)
Other:
- moved on the sheet: C12, R10, R5
